File: hardware/pcb/projects/igb01_led/igb01_led.kicad_sch (KiCad schematic)
At the start: 18 parts, among them J1 LED_CON_L, J2 LED_CON_R

Commit message: update led board
Parts:
- removed J1: LED_CON_L, symbol Connector_Generic:Conn_01x10
- removed J2: LED_CON_R, symbol Connector_Generic:Conn_01x10
- added C1, C3, C4: 100n, Capacitor_SMD:C_0402_1005Metric, symbol Device:C_Small
- added C2: 100u, Capacitor_THT:CP_Radial_D6.3mm_P2.50mm, symbol Device:C_Polarized
- added D17, D18, D20, D61, D62, D63, D64, D65, D66, D67, D68, D69, D70, D71, D72, D73, D74, D75, D76, D85, D86, D87, D88, D89, D90, D91, D92, D93, D94, D95, D96: GreenS, custom:LED_Kingbright_APA2106, symbol Device:LED_Small
- added D19: RedS, custom:LED_Kingbright_APA2106, symbol Device:LED_Small
- added D21, D23, D25, D27, D29, D31, D33, D35, D37, D39, D41, D43, D45, D47, D49, D51: Red, LED_SMD:LED_0603_1608Metric, symbol Device:LED_Small
- added D22, D24, D26, D28, D30, D32, D34, D36, D38, D40, D42, D44, D46, D48, D50, D52, D53, D54, D55, D56, D57, D58, D59, D60, D77, D78, D79, D80, D81, D82, D83, D84: Green, LED_SMD:LED_0603_1608Metric, symbol Device:LED_Small
- added J1: ConnToCtrl, Connector_PinSocket_2.00mm:PinSocket_1x04_P2.00mm_Vertical, symbol Connector_Generic:Conn_01x04
- added J2, J3, J5, J6: Hold_Conn, Connector_PinSocket_2.00mm:PinSocket_1x03_P2.00mm_Vertical, symbol Connector_Generic:Conn_01x03
- added J4: GND_Conn, Connector_PinSocket_2.00mm:PinSocket_1x03_P2.00mm_Vertical, symbol Connector_Generic:Conn_01x03
- added R1: 100k, Resistor_SMD:R_0603_1608Metric, symbol Device:R
- added R2: 10k, Resistor_SMD:R_0603_1608Metric, symbol Device:R
- added R3: 47k, Resistor_SMD:R_0603_1608Metric, symbol Device:R
- added U1: IS31FL3731-QF, Package_DFN_QFN:QFN-28-1EP_4x4mm_P0.4mm_EP2.3x2.3mm, symbol Driver_LED:IS31FL3731-QF
- renumbered D4 to D10, D6 to D11, D8 to D12, D10 to D13, D12 to D14, D14 to D15, D3 to D2, D5 to D3, D7 to D4, D9 to D5, D11 to D6, D13 to D7, D15 to D8, D2 to D9
Connections:
- net GND: now also C1.2, C2.2, C3.2, C4.2, J1.1 (Pin_1), J4.1 (Pin_1), J4.2 (Pin_2), J4.3 (Pin_3), R3.2, U1.29 (GND), U1.5 (GND)
- net at D1.4 (RK), D10.1 (BK), D12.1 (BK)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: now also D20.2 (A), D27.2 (A), D28.1 (K), U1.24 (CA4)
- net at D10.4 (RK), D12.4 (RK), D13.2 (A)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: now also D33.2 (A), D34.1 (K), U1.27 (CA7)
- net at D10.2 (A), D12.3 (GK), D14.3 (GK)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: now also D29.2 (A), D30.1 (K), U1.25 (CA5)
- net at D10.3 (GK), D11.2 (A), D12.2 (A)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: now also D31.2 (A), D32.1 (K), U1.26 (CA6)
- net at D1.2 (A), D11.1 (BK), D13.1 (BK)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: now also D17.2 (A), D21.2 (A), D22.1 (K), U1.21 (CA1)
- net at D1.3 (GK), D11.4 (RK), D13.4 (RK)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: now also D19.2 (A), D25.2 (A), D26.1 (K), U1.23 (CA3)
- net at D1.1 (BK), D11.3 (GK), D13.3 (GK)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: now also D18.2 (A), D23.2 (A), D24.1 (K), U1.22 (CA2)
- net at D15.2 (A), D16.2 (A): now also D17.1 (K), D18.1 (K), D19.1 (K), D20.1 (K), D35.2 (A), D36.1 (K), U1.28 (CA8)
- new net: D57.1 (K), D58.2 (A), D59.1 (K), D60.2 (A), D61.1 (K), D62.2 (A), D63.1 (K), D64.2 (A), D75.2 (A), D76.1 (K), D87.2 (A), D88.1 (K), U1.12 (CB6)
- new net: D41.1 (K), D42.2 (A), D47.1 (K), D48.2 (A), D51.1 (K), D52.2 (A), D55.2 (A), D56.1 (K), D61.2 (A), D62.1 (K), D71.2 (A), D72.1 (K), D83.2 (A), D84.1 (K), U1.10 (CB4)
- new net: D65.1 (K), D66.2 (A), D67.1 (K), D68.2 (A), D69.1 (K), D70.2 (A), D71.1 (K), D72.2 (A), D73.1 (K), D74.2 (A), D75.1 (K), D76.2 (A), D89.2 (A), D90.1 (K), U1.13 (CB7)
- new net: D43.1 (K), D44.2 (A), D49.1 (K), D50.2 (A), D53.1 (K), D54.2 (A), D55.1 (K), D56.2 (A), D63.2 (A), D64.1 (K), D73.2 (A), D74.1 (K), D85.2 (A), D86.1 (K), U1.11 (CB5)
- new net: D37.1 (K), D38.2 (A), D45.2 (A), D46.1 (K), D47.2 (A), D48.1 (K), D49.2 (A), D50.1 (K), D59.2 (A), D60.1 (K), D67.2 (A), D68.1 (K), D79.2 (A), D80.1 (K), D93.2 (A), D94.1 (K), U1.8 (CB2)
- new net: D37.2 (A), D38.1 (K), D39.2 (A), D40.1 (K), D41.2 (A), D42.1 (K), D43.2 (A), D44.1 (K), D57.2 (A), D58.1 (K), D65.2 (A), D66.1 (K), D77.2 (A), D78.1 (K), D91.2 (A), D92.1 (K), U1.7 (CB1)
- new net: D91.1 (K), D92.2 (A), D93.1 (K), D94.2 (A), D95.1 (K), D96.2 (A), U1.15 (CB9)
- new net: D77.1 (K), D78.2 (A), D79.1 (K), D80.2 (A), D81.1 (K), D82.2 (A), D83.1 (K), D84.2 (A), D85.1 (K), D86.2 (A), D87.1 (K), D88.2 (A), D89.1 (K), D90.2 (A), U1.14 (CB8)
- new net: D39.1 (K), D40.2 (A), D45.1 (K), D46.2 (A), D51.2 (A), D52.1 (K), D53.2 (A), D54.1 (K), D69.2 (A), D70.1 (K), D81.2 (A), D82.1 (K), D95.2 (A), D96.1 (K), U1.9 (CB3)
- new net: D21.1 (K), D22.2 (A), D23.1 (K), D24.2 (A), D25.1 (K), D26.2 (A), D27.1 (K), D28.2 (A), D29.1 (K), D30.2 (A), D31.1 (K), D32.2 (A), D33.1 (K), D34.2 (A), D35.1 (K), D36.2 (A), U1.1 (CA9)
- new net: C4.1, U1.16 (C_FILT)
- new net: C3.1, U1.17 (IN)
- new net: R1.2, U1.3 (~{SDB})
- new net: R3.1, U1.6 (R_EXT)
- new net +3.3V: C1.1, C2.1, J1.4 (Pin_4), R1.1, R2.1, U1.18 (AD), U1.2 (VCC)
- new net INTB: R2.2, U1.4 (~{INTB})
- new net SCL: J1.3 (Pin_3), U1.20 (SCL)
- new net SDA: J1.2 (Pin_2), U1.19 (SDA)
- no-connect marks 0 -> 12
Other:
- note added: "C1-10 C3-9"
- note added: "C1-11 C4-9"
- note added: "C1-12 C5-9"
- note added: "C1-13"
- note added: "C1-14"
- note added: "C1-15"
- note added: "C1-16"
- note added: "C1-9 C2-9"
- note added: "C2-10 C3-10"
- note added: "C2-11 C4-10"
- note added: "C2-12 C5-10"
- note added: "C2-13"
- note added: "C2-14"
- note added: "C2-15"
- note added: "C2-16"
- note added: "C3-11 C4-11"
- note added: "C3-12"
- note added: "C3-14"
- note added: "C3-15"
- note added: "C3-16"
- note added: "C4-12"
- note added: "C4-13"
- note added: "C4-14"
- note added: "C4-15"
- note added: "C5-11"
- note added: "C5-12"
- note added: "C5-13"
- note added: "C5-14"
- note added: "C5-15"
- note added: "C6-10"
- note added: "C6-12"
- note added: "C6-13"
- note added: "C6-14"
- note added: "C6-15"
- note added: "C6-9"
- note added: "C7-10"
- note added: "C7-11"
- note added: "C7-12"
- note added: "C7-13"
- note added: "C7-14"
- note added: "C7-15"
- note added: "C7-9"
- note added: "C8-1"
- note added: "C8-10"
- note added: "C8-11"
- note added: "C8-12"
- note added: "C8-13"
- note added: "C8-14"
- note added: "C8-15"
- note added: "C8-2"
- note added: "C8-3"
- note added: "C8-4"
- note added: "C8-9"
- note added: "C9-1 C1-8"
- note added: "C9-10"
- note added: "C9-11"
- note added: "C9-2 C2-8"
- note added: "C9-3 C3-8"
- note added: "C9-4 C4-8"
- note added: "C9-5 C5-8"
- note added: "C9-6 C6-8"
- note added: "C9-7 C7-8"
- note added: "C9-8 C8-8"
- note added: "C9-9"
- note added: "FINE/SELECT/REC/PLAY LEDs"
- note added: "KEYBOARD Buttons"
- note added: "LED Driver"
- note added: "Macro Knob Button LEDs"
- note added: "Mixer Level LEDs"
- note added: "OCTAVE Buttons"
- note added: "PATTERN/TRACK LEDs"
- note added: "Ribbon Mode LEDs"
- note added: "Side View LED Red: APA2106SURCK (C5553569) Side View LED Green: APA2106ZGC (C5879337)"
- note added: "TOUCH LEDs"
- note added: "back side mount"
- note removed: "CA1"
- note removed: "CA2"
- note removed: "CA3"
- note removed: "CA4"
- note removed: "CA5"
- note removed: "CA6"
- note removed: "CA7"
- note removed: "CA8"
- note removed: "CA9"
- note removed: "Touch Pad Board Connector"
- moved on the sheet: D1, D10, D11, D12, D13, D14, D15, D16, D2, D3, D4, D5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

Commit message: update igb01 led pcb
Parts:
- added C10: 10u, Capacitor_SMD:C_0402_1005Metric, symbol Device:C_Small
- added C11: 1n, Capacitor_SMD:C_0402_1005Metric, symbol Device:C_Small
- added C12, C13: 18p, Capacitor_SMD:C_0402_1005Metric, symbol Device:C_Small
- added C14, C15, C16, C17, C18, C19: 22n, Capacitor_SMD:C_0402_1005Metric, symbol Device:C_Small
- added C20, C6, C7, C8, C9: 100n, Capacitor_SMD:C_0402_1005Metric, symbol Device:C_Small
- added C5: 100u, Capacitor_SMD:CP_Elec_6.3x5.2, symbol Device:C_Polarized
- added D101, D102, D103, D104, D105, D106, D107, D108, D109, D110, D63, D64: GreenS, custom:LED_Kingbright_APA2106, symbol Device:LED_Small
- added D21: Red, LED_SMD:LED_0603_1608Metric, symbol Device:LED_Small
- added D22: Green, LED_SMD:LED_0603_1608Metric, symbol Device:LED_Small
- added J10, J11, J12, J9: TOUCH_CONN, custom:CONN_47286-1001_MOL, symbol Connector_Generic:Conn_01x04
- added J13: PositionSensorCon, Connector_PinSocket_2.54mm:PinSocket_1x03_P2.54mm_Horizontal, symbol Connector_Generic:Conn_01x03
- added J7: McuConn, Connector_PinSocket_2.00mm:PinSocket_1x04_P2.00mm_Vertical, symbol Connector_Generic:Conn_01x06
- added J8: SWD, Connector_PinSocket_2.54mm:PinSocket_1x05_P2.54mm_Horizontal, symbol Connector_Generic:Conn_01x05
- added R10, R11, R12, R13, R14, R15, R16, R17, R18, R19, R20, R21, R6, R7, R8, R9: 470, Resistor_SMD:R_0603_1608Metric, symbol Device:R
- added R22, R23: 1k, Resistor_SMD:R_0603_1608Metric, symbol Device:R
- added R24: 120k, Resistor_SMD:R_0603_1608Metric, symbol Device:R
- added R25, R27: 100k, Resistor_SMD:R_0603_1608Metric, symbol Device:R
- added R26, R28: 470k, Resistor_SMD:R_0603_1608Metric, symbol Device:R
- added R29: 10M, Resistor_SMD:R_0603_1608Metric, symbol Device:R
- added R4, R5: 10k, Resistor_SMD:R_0603_1608Metric, symbol Device:R
- added TP1, TP2: TestPoint, TestPoint:TestPoint_Pad_1.0x1.0mm, symbol Connector:TestPoint
- added U2: STM32F303RBTx, Package_QFP:LQFP-64_10x10mm_P0.5mm, symbol MCU_ST_STM32F3:STM32F303RBTx
- added U3: MCP6002-xMS, Package_SO:MSOP-8_3x3mm_P0.65mm, symbol Amplifier_Operational:MCP6002-xMS
- added Y1: 12MHz, Crystal:Crystal_SMD_2520-4Pin_2.5x2.0mm, symbol Device:Crystal_GND24_Small
- C2: footprint Capacitor_THT:CP_Radial_D6.3mm_P2.50mm -> Capacitor_SMD:CP_Elec_6.3x5.2
- J1: value ConnToCtrl -> LedDrvConn
- renumbered D96 to D100, D21 to D23, D22 to D24, D23 to D25, D24 to D26, D25 to D27, D26 to D28, D27 to D29, D28 to D30, D29 to D31, D30 to D32, D31 to D33, D32 to D34, D33 to D35, D34 to D36, D35 to D37, D36 to D38, D37 to D39, D38 to D40, D39 to D41, D40 to D42, D41 to D43, D42 to D44, D43 to D45, D44 to D46, D45 to D47, D46 to D48, D47 to D49, D48 to D50, D49 to D51, D50 to D52, D51 to D53, D52 to D54, D53 to D55, D54 to D56, D55 to D57, D56 to D58, D57 to D59, D58 to D60, D59 to D61, D60 to D62, D61 to D65, D62 to D66, D63 to D67, D64 to D68, D65 to D69, D66 to D70, D67 to D71, D68 to D72, D69 to D73, D70 to D74, D71 to D75, D72 to D76, D73 to D77, D74 to D78, D75 to D79, D76 to D80, D77 to D81, D78 to D82, D79 to D83, D80 to D84, D81 to D85, D82 to D86, D83 to D87, D84 to D88, D85 to D89, D86 to D90, D87 to D91, D88 to D92, D89 to D93, D90 to D94, D91 to D95, D92 to D96, D93 to D97, D94 to D98, D95 to D99, J4 to J2, J2 to J3, J5 to J4, J3 to J5
Connections:
- net +3.3V: now also C5.1, C6.1, C7.1, C8.1, C9.1, J7.4 (Pin_4), J8.1 (Pin_1), R4.1, U2.19 (VDD), U2.32 (VDD), U2.48 (VDD), U2.64 (VDD); no longer C1.1, C2.1, J1.4 (Pin_4), U1.2 (VCC)
- net GND: now also J1.2 (Pin_2); no longer J1.1 (Pin_1)
- net at D59.1 (K), D60.2 (A), D61.1 (K)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: now also D105.2 (A), D106.1 (K), D63.1 (K), D64.2 (A)
- net at D43.1 (K), D44.2 (A), D49.1 (K)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: now also D101.2 (A), D102.1 (K)
- net at D69.1 (K), D70.2 (A), D71.1 (K)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: now also D107.2 (A), D108.1 (K)
- net at D15.2 (A), D16.2 (A), D17.1 (K)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: now also D21.1 (K), D22.1 (K)
- net at D45.1 (K), D46.2 (A), D51.1 (K)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: now also D103.2 (A), D104.1 (K)
- net at D10.2 (A), D12.3 (GK), D14.3 (GK)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: now also D21.2 (A)
- net at D10.3 (GK), D11.2 (A), D12.2 (A)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: now also D22.2 (A)
- net at D100.2 (A), D95.1 (K), D96.2 (A)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: now also D101.1 (K), D102.2 (A), D103.1 (K), D104.2 (A), D105.1 (K), D106.2 (A), D107.1 (K), D108.2 (A), D109.1 (K), D110.2 (A)
- net at D81.1 (K), D82.2 (A), D83.1 (K)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: now also D109.2 (A), D110.1 (K)
- net at D100.1 (K), D41.1 (K), D42.2 (A)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: now also D63.2 (A), D64.1 (K)
- net SCL renamed LED_DRV_SCL
- net SDA renamed LED_DRV_SDA
- net LED_DRV_SDA: now also J1.1 (Pin_1); no longer J1.2 (Pin_2)
- new net: R25.2, R26.2, U3.5 (+)
- new net: R27.2, R28.1, U3.6 (-)
- new net: C12.2, U2.5 (PF0), Y1.3
- new net: J13.2 (Pin_2), R29.2, U3.3 (+)
- new net: J12.4 (Pin_4), R21.2
- new net: J12.2 (Pin_2), R13.2
- new net: J11.2 (Pin_2), R12.2
- new net: J13.3 (Pin_3), R22.1, R25.1
- new net: J10.3 (Pin_3), R15.2
- new net: R23.1, R24.2, R27.1
- new net: J11.4 (Pin_4), R20.2
- new net: J9.3 (Pin_3), R14.2
- new net: J12.1 (Pin_1), R9.2
- new net: J10.2 (Pin_2), R11.2
- new net: R5.2, U2.60 (BOOT0)
- new net: J12.3 (Pin_3), R17.2
- new net: J9.1 (Pin_1), R6.2
- new net: J9.2 (Pin_2), R10.2
- new net: J9.4 (Pin_4), R18.2
- new net: C13.2, U2.6 (PF1), Y1.1
- new net: J11.3 (Pin_3), R16.2
- new net: J10.1 (Pin_1), R7.2
- new net: J10.4 (Pin_4), R19.2
- new net: J11.1 (Pin_1), R8.2
- new net +3.3VA: C10.1, C11.1, C20.1, J13.1 (Pin_1), J7.5 (Pin_5), R24.1, U2.13 (VDDA), U3.8 (V+)
- new net +3.3VP: C1.1, C2.1, J1.4 (Pin_4), U1.2 (VCC)
- new net GND1: C10.2, C11.2, C12.1, C13.1, C14.2, C15.2, C16.2, C17.2, C18.2, C19.2, C5.2, C6.2, C7.2, C8.2, C9.2, J7.2 (Pin_2), J8.3 (Pin_3), R5.1, U2.31 (VSS), U2.47 (VSS), U2.63 (VSS), Y1.2, Y1.4
- new net GNDA: C20.2, J7.6 (Pin_6), R22.2, R23.2, R26.1, R29.1, U2.12 (VSSA), U3.4 (V-)
- new net MCU_ADC_POS: TP1.1, U2.17 (PA3), U3.1, U3.2 (-)
- new net MCU_ADC_PRES: R28.2, TP2.1, U2.16 (PA2), U3.7
- new net MCU_SCL: J7.3 (Pin_3), U2.61 (PB8)
- new net MCU_SDA: J7.1 (Pin_1), U2.62 (PB9)
- new net MCU_SWCLK: J8.2 (Pin_2), R12.1, U2.49 (PA14)
- new net MCU_SWDIO: J8.4 (Pin_4), R8.1, U2.46 (PA13)
- new net TSC_G1_IO1: C14.1, U2.14 (PA0)
- new net TSC_G1_IO2: R6.1, U2.15 (PA1)
- new net TSC_G2_IO1: C15.1, U2.20 (PA4)
- new net TSC_G2_IO2: R10.1, U2.21 (PA5)
- new net TSC_G2_IO3: R14.1, U2.22 (PA6)
- new net TSC_G2_IO4: R18.1, U2.23 (PA7)
- new net TSC_G3_IO1: C16.1, U2.25 (PC5)
- new net TSC_G3_IO2: R7.1, U2.26 (PB0)
- new net TSC_G3_IO3: R11.1, U2.27 (PB1)
- new net TSC_G3_IO4: R15.1, U2.28 (PB2)
- new net TSC_G4_IO1: C17.1, U2.42 (PA9)
- new net TSC_G4_IO2: R19.1, U2.43 (PA10)
- new net TSC_G5_IO1: C18.1, U2.55 (PB3)
- new net TSC_G5_IO2: R16.1, U2.56 (PB4)
- new net TSC_G5_IO3: R20.1, U2.58 (PB6)
- new net TSC_G5_IO4: R9.1, U2.59 (PB7)
- new net TSC_G6_IO1: C19.1, U2.30 (PB11)
- new net TSC_G6_IO2: R13.1, U2.33 (PB12)
- new net TSC_G6_IO3: R17.1, U2.34 (PB13)
- new net TSC_G6_IO4: R21.1, U2.35 (PB14)
- new net ~{MCU_RESET}: J8.5 (Pin_5), R4.2, U2.7 (NRST)
- no-connect marks 12 -> 37
Other:
- note added: "C3-13"
- note added: "C4-16"
- note added: "C5-16"
- note added: "C6-11"
- note added: "C6-16"
- note added: "C7-16"
- note added: "C8-16"
- note added: "C8-5"
- note added: "C8-6"
- note added: "C9-12"
- note added: "C9-13"
- note added: "C9-14"
- note added: "C9-15"
- note added: "C9-16"
- note added: "LEVEL LEDs"
- note added: "Sping Connector: Molex 0472861001 (https://www.molex.com/en-us/products/part-detail/472861001)"
- note added: "TODO: 16 touch pad (TSC) & Position Sensor Pot (Position ADC IN/ Pressure ADC IN)"
- note added: "TSC_G4_IO3"
- note added: "TSC_G4_IO4"
- note added: "Touch Slider LEDs"
- moved on the sheet: D100, D65, D66, D67, D68, D69, D70, D71, D72, D73, D74, D75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

Commit message: update led schematic
Parts:
- added R30, R31, R32, R33, R34, R35: 10, Resistor_SMD:R_0603_1608Metric, symbol Device:R
Connections:
- net LED_DRV_SCL: now also R31.2, R32.1; no longer U1.20 (SCL)
- net LED_DRV_SDA: now also R30.2, R33.1; no longer U1.19 (SDA)
- net at U2.51 (PC10): now also R34.2
- net at U2.52 (PC11): now also R35.2
- net MCU_SCL: no longer names the net of U2.61 (PB8)
- net MCU_SCL: now also R32.2; no longer J7.3 (Pin_3)
- net MCU_SDA: no longer names the net of U2.62 (PB9)
- net MCU_SDA: now also R33.2; no longer J7.1 (Pin_1)
- new net: R30.1, U1.19 (SDA)
- new net: R31.1, U1.20 (SCL)
- new net USART3_RX: J7.3 (Pin_3), R35.1
- new net USART3_TX: J7.1 (Pin_1), R34.1
- no-connect marks 37 -> 35

Commit message: update led&control schematics
Parts:
- added J14: Hold_Conn, Connector_PinSocket_2.00mm:PinSocket_1x03_P2.00mm_Vertical, symbol Connector_Generic:Conn_01x03
- J1: footprint Connector_PinSocket_2.00mm:PinSocket_1x04_P2.00mm_Vertical -> Connector_PinSocket_2.00mm:PinSocket_1x06_P2.00mm_Vertical; symbol Connector_Generic:Conn_01x04 -> Connector_Generic:Conn_01x06
- J2: value GND_Conn -> Hold_Conn
Connections:
- net +3.3V: no longer R1.1, R2.1
- net +3.3VP: now also J1.5 (Pin_5), J1.6 (Pin_6), R1.1, R2.1; no longer J1.4 (Pin_4)
- net GND: now also J1.3 (Pin_3); no longer J2.1 (Pin_1), J2.2 (Pin_2), J2.3 (Pin_3)
- net LED_DRV_SCL: now also J1.4 (Pin_4); no longer J1.3 (Pin_3)
- no-connect marks 35 -> 41
