File: hardware/pcb/projects/igb01_core/igb01_core.kicad_sch (KiCad schematic)
At the start: 100 parts, among them J1 STMP157_GPIO1, J10 I2C_PREV, J11 I2C_NEXT, J12 STMP157_GPIO3, J13 JTAG, J14 USB_CONN, J15 STMP157_GPIO4, J16 Micro_SD_Card, J17 PWR_ON_CON, J18 STMP157_GPIO5, J19 STMP157_GPIO6, J2 BAT_CON, J20 FPA-VZA2-15-LF, J22 Conn_01x13, J3 VBUS_CON, J4 LEFT_CON, J5 RIGHT_CON, J6 STMP157_GPIO2, J7 IGB2_NEXT, J8 IGB3_NEXT, J9 IGB4_NEXT, SW1 SW_DIP_x04, SW2 SW_Push, SW3 SW_Push, U1 W25Q128JVS, U2 AK4619

Commit message: update core board sch&pcb
Parts:
- removed C3: 47u, Resistor_SMD:R_1206_3216Metric, symbol Device:C_Small
- removed R18, R19, R22, R25: 10k, Resistor_SMD:R_0603_1608Metric, symbol Device:R
- added C19: 100n, Capacitor_SMD:C_0402_1005Metric, symbol Device:C_Small
- added J6: IGB2_PREV, Connector_Molex:Molex_KK-254_AE-6410-03A_1x03_P2.54mm_Vertical, symbol Connector_Generic:Conn_01x03
- added R14, R15, R16, R17, R2, R3: 22, Resistor_SMD:R_0603_1608Metric, symbol Device:R
- added R41, R42: 22, Resistor_SMD:R_0402_1005Metric, symbol Device:R
- added R47, R48: 10k, Resistor_SMD:R_0402_1005Metric, symbol Device:R
- added R51: 10k, Resistor_SMD:R_0603_1608Metric, symbol Device:R
- C1: footprint Resistor_SMD:R_1206_3216Metric -> Capacitor_SMD:C_1206_3216Metric
- C10, C11, C12, C20, C21, C22, C23, C9: footprint Capacitor_SMD:C_1206_3216Metric -> Capacitor_SMD:C_0805_2012Metric
- C2: footprint Resistor_SMD:R_1206_3216Metric -> Capacitor_SMD:C_0805_2012Metric
- C3: renamed from C4; footprint Resistor_SMD:R_1206_3216Metric -> Capacitor_SMD:C_1206_3216Metric
- C4: renamed from C5; value 100n -> 47u; footprint Resistor_SMD:R_0603_1608Metric -> Capacitor_SMD:C_0805_2012Metric
- C5: renamed from C6; footprint Resistor_SMD:R_1206_3216Metric -> Capacitor_SMD:C_0805_2012Metric
- C7: renamed from C16; footprint Resistor_SMD:R_1206_3216Metric -> Capacitor_SMD:C_0805_2012Metric
- R18: renamed from R12; value 10k -> 47k; footprint Resistor_SMD:R_0603_1608Metric -> Resistor_SMD:R_0402_1005Metric
- R19: renamed from R13; value 10k -> 47k; footprint Resistor_SMD:R_0603_1608Metric -> Resistor_SMD:R_0402_1005Metric
- R20: renamed from R14; value 10k -> 47k; footprint Resistor_SMD:R_0603_1608Metric -> Resistor_SMD:R_0402_1005Metric
- R21: renamed from R15; value 10k -> 47k; footprint Resistor_SMD:R_0603_1608Metric -> Resistor_SMD:R_0402_1005Metric
- R23: renamed from R17; value 10k -> 47k; footprint Resistor_SMD:R_0603_1608Metric -> Resistor_SMD:R_0402_1005Metric
- R24: renamed from R20; value 10k -> 47k; footprint Resistor_SMD:R_0603_1608Metric -> Resistor_SMD:R_0402_1005Metric
- R25: renamed from R21; value 10k -> 47k; footprint Resistor_SMD:R_0603_1608Metric -> Resistor_SMD:R_0402_1005Metric
- R26: renamed from R23; value 10k -> 47k; footprint Resistor_SMD:R_0603_1608Metric -> Resistor_SMD:R_0402_1005Metric
- R27: renamed from R24; value 10k -> 47k; footprint Resistor_SMD:R_0603_1608Metric -> Resistor_SMD:R_0402_1005Metric
- R28: renamed from R26; value 10k -> 47k; footprint Resistor_SMD:R_0603_1608Metric -> Resistor_SMD:R_0402_1005Metric
- R29: renamed from R27; footprint Resistor_SMD:R_0603_1608Metric -> Resistor_SMD:R_0402_1005Metric
- R30: renamed from R28; footprint Resistor_SMD:R_0603_1608Metric -> Resistor_SMD:R_0402_1005Metric
- R31: renamed from R29; footprint Resistor_SMD:R_0603_1608Metric -> Resistor_SMD:R_0402_1005Metric
- R32: renamed from R30; footprint Resistor_SMD:R_0603_1608Metric -> Resistor_SMD:R_0402_1005Metric
- R33: renamed from R31; footprint Resistor_SMD:R_0603_1608Metric -> Resistor_SMD:R_0402_1005Metric
- R34: renamed from R32; footprint Resistor_SMD:R_0603_1608Metric -> Resistor_SMD:R_0402_1005Metric
- R35: renamed from R33; footprint Resistor_SMD:R_0603_1608Metric -> Resistor_SMD:R_0402_1005Metric
- R36: renamed from R34; footprint Resistor_SMD:R_0603_1608Metric -> Resistor_SMD:R_0402_1005Metric
- R4: renamed from R2; value 47 -> 22
- R49: renamed from R47; footprint Resistor_SMD:R_0603_1608Metric -> Resistor_SMD:R_0402_1005Metric
- R5: renamed from R3; value 47 -> 22
- R50: renamed from R48; footprint Resistor_SMD:R_0603_1608Metric -> Resistor_SMD:R_0402_1005Metric
- R6: renamed from R4; value 47 -> 22
- R7: renamed from R5; value 47 -> 22
- R8: renamed from R6; value 47 -> 22
- R9: renamed from R7; value 47 -> 22
- renumbered C17 to C16, C18 to C17, C19 to C18, C7 to C6, J2 to J1, J6 to J12, J14 to J13, J12 to J14, J13 to J15, J15 to J16, J16 to J17, J17 to J18, J18 to J19, J3 to J2, J19 to J21, J1 to J3, R8 to R10, R9 to R11, R10 to R12, R11 to R13, R16 to R22, R35 to R37, R36 to R38, R37 to R39, R42 to R40, R38 to R52, R39 to R53, R40 to R54, R41 to R55
Connections:
- net +3.3V: now also R47.2, R48.2
- net +3.3VA: now also C17.1, C18.1, U2.21 (VREFH)
- net CODEC_PDN: now also C19.1, R51.2
- net GND: now also J10.2 (Pin_2), J11.2 (Pin_2), J4.6 (Pin_6), J4.7 (Pin_7), J7.2 (Pin_2), J8.2 (Pin_2), J9.2 (Pin_2), C19.2, J6.2 (Pin_2), R51.1; no longer J10.1 (Pin_1), J11.1 (Pin_1), J7.1 (Pin_1), J8.1 (Pin_1), J9.1 (Pin_1), U2.2 (SDIN2), U2.27 (I2CAD/CS)
- net IN1L: now also J5.8 (Pin_8); no longer J5.3 (Pin_3)
- net IN1R: now also J5.9 (Pin_9); no longer J5.4 (Pin_4)
- net IN2L: now also J5.10 (Pin_10); no longer J5.5 (Pin_5)
- net IN2R: now also J5.11 (Pin_11); no longer J5.6 (Pin_6)
- net OUT1L: now also J5.6 (Pin_6); no longer J5.8 (Pin_8)
- net OUT1R: now also J5.5 (Pin_5); no longer J5.9 (Pin_9)
- net OUT2L: now also J5.4 (Pin_4); no longer J5.10 (Pin_10)
- net OUT2R: now also J5.3 (Pin_3); no longer J5.11 (Pin_11)
- net USART4_RX: now also R2.2; no longer J4.6 (Pin_6)
- net USART4_TX: now also R3.2; no longer J4.7 (Pin_7)
- net USB1_D+: now also R14.2; no longer J13.1 (Pin_1)
- net USB1_D-: now also R15.2; no longer J13.2 (Pin_2)
- net USB_OTG_FS_D+: now also R16.2; no longer J13.5 (Pin_5)
- net USB_OTG_FS_D-: now also R17.2; no longer J13.6 (Pin_6)
- net at R4.1: now also J7.1 (Pin_1); no longer J7.2 (Pin_2)
- net at R8.1: now also J9.1 (Pin_1); no longer J9.2 (Pin_2)
- net  SAI1_SD_B: now reaches J16.10 (Pin_10)
- net  SAI1_SD_B: now also R41.1
- net at R6.1: now also J8.1 (Pin_1); no longer J8.2 (Pin_2)
- net at U2.29 (MOSI): now also R47.1
- net at U2.32 (SDOUT2): now also R42.1
- net at R10.1: now also J10.1 (Pin_1); no longer J10.2 (Pin_2)
- net at R12.1: now also J11.1 (Pin_1); no longer J11.2 (Pin_2)
- net SAI1_SD_A: now reaches J12.24 (Pin_24)
- net SAI1_SD_A: now also R42.2
- net EXT_GPIO0: no longer names the net of J21.7 (Pin_7)
- net EXT_GPIO1: no longer names the net of J21.9 (Pin_9)
- net EXT_GPIO2: no longer names the net of J21.11 (Pin_11)
- net EXT_GPIO3: no longer names the net of J21.13 (Pin_13)
- net EXT_GPIO4: no longer names the net of J21.15 (Pin_15)
- net EXT_GPIO5: no longer names the net of J21.14 (Pin_14)
- net EXT_GPIO6: no longer names the net of J21.22 (Pin_22)
- net EXT_GPIO7: no longer names the net of J21.24 (Pin_24)
- new net: J13.1 (Pin_1), R14.1
- new net: J13.2 (Pin_2), R15.1
- new net: J13.5 (Pin_5), R16.1
- new net: J13.6 (Pin_6), R17.1
- new net: R41.2, U2.2 (SDIN2)
- new net: R48.1, U2.27 (I2CAD/CS)
- new net: J6.1 (Pin_1), R2.1
- new net: J6.3 (Pin_3), R3.1
- no-connect marks 110 -> 114
Other:
- note added: "+2.8V"
- note added: "1.2V_HDMI"
- note added: "ADC1_INN1"
- note added: "AXP_BACKUP"
- note added: "AXP_EXTEN"
- note added: "AXP_GPIO0"
- note added: "AXP_GPIO1"
- note added: "AXP_GPIO2/LCD_LR"
- note added: "AXP_GPIO3/LCD_UD"
- note added: "PA1/GRXD_CLK"
- note added: "PA13"
- note added: "PA14"
- note added: "PA15"
- note added: "PA2"
- note added: "PA3"
- note added: "PA4"
- note added: "PA5"
- note added: "PA6"
- note added: "PA7/GRXD_DV"
- note added: "PA8"
- note added: "PA9"
- note added: "PB0/GRXD2"
- note added: "PB1/GRXD3"
- note added: "PB10"
- note added: "PB11/GTXD_EN"
- note added: "PB12"
- note added: "PB13"
- note added: "PB14"
- note added: "PB15"
- note added: "PB3"
- note added: "PB4"
- note added: "PB5"
- note added: "PB6"
- note added: "PB7"
- note added: "PB8"
- note added: "PB9"
- note added: "PC0"
- note added: "PC1"
- note added: "PC10"
- note added: "PC11"
- note added: "PC12"
- note added: "PC13"
- note added: "PC2/GTXD2"
- note added: "PC3"
- note added: "PC4/GRXD0"
- note added: "PC5/GRXD1"
- note added: "PC6"
- note added: "PC7"
- note added: "PC8"
- note added: "PC9"
- note added: "PD0"
- note added: "PD1"
- note added: "PD10"
- note added: "PD11"
- note added: "PD12"
- note added: "PD13"
- note added: "PD14"
- note added: "PD15"
- note added: "PD2"
- note added: "PD3"
- note added: "PD4"
- note added: "PD5"
- note added: "PD6"
- note added: "PD7"
- note added: "PD8"
- note added: "PD9"
- note added: "PE0"
- note added: "PE1"
- note added: "PE10"
- note added: "PE11"
- note added: "PE12"
- note added: "PE13"
- note added: "PE14"
- note added: "PE15"
- note added: "PE2/GTXD3"
- note added: "PE3"
- note added: "PE4"
- note added: "PE5"
- note added: "PE6"
- note added: "PE7"
- note added: "PE8"
- note added: "PE9"
- note added: "PF0"
- note added: "PF1"
- note added: "PF10"
- note added: "PF11"
- note added: "PF12"
- note added: "PF13"
- note added: "PF14"
- note added: "PF15"
- note added: "PF2"
- note added: "PF3"
- note added: "PF4"
- note added: "PF5"
- note added: "PF6"
- note added: "PF7"
- note added: "PF8"
- note added: "PF9"
- note added: "PG0"
- note added: "PG1"
- note added: "PG10"
- note added: "PG11"
- note added: "PG12"
- note added: "PG13/GTXD0"
- note added: "PG14/GTXD1"
- note added: "PG15"
- note added: "PG2"
- note added: "PG3"
- note added: "PG4/GTXD_CLK"
- note added: "PG5"
- note added: "PG6"
- note added: "PG7"
- note added: "PG8"
- note added: "PG9"
- note added: "PH10"
- note added: "PH11"
- note added: "PH12"
- note added: "PH13"
- note added: "PH14"
- note added: "PH15"
- note added: "PH2"
- note added: "PH3"
- note added: "PH4"
- note added: "PH5"
- note added: "PH6"
- note added: "PH7"
- note added: "PH8"
- note added: "PH9"
- note added: "PI0"
- note added: "PI1"
- note added: "PI10"
- note added: "PI11"
- note added: "PI12"
- note added: "PI13"
- note added: "PI14"
- note added: "PI15"
- note added: "PI2"
- note added: "PI3"
- note added: "PI4"
- note added: "PI5"
- note added: "PI6"
- note added: "PI7"
- note added: "PI8"
- note added: "PI9"
- note added: "PJ0"
- note added: "PJ1"
- note added: "PJ10"
- note added: "PJ11"
- note added: "PJ12"
- note added: "PJ13"
- note added: "PJ14"
- note added: "PJ15"
- note added: "PJ2"
- note added: "PJ3"
- note added: "PJ4"
- note added: "PJ5"
- note added: "PJ6"
- note added: "PJ7"
- note added: "PJ8"
- note added: "PJ9"
- note added: "PK0"
- note added: "PK1"
- note added: "PK2"
- note added: "PK3"
- note added: "PK4"
- note added: "PK5"
- note added: "PK6"
- note added: "PK7"
- note added: "PZ0"
- note added: "PZ1"
- note added: "PZ2"
- note added: "PZ3"
- note added: "PZ4"
- note added: "PZ5"
- note added: "PZ6"
- note added: "PZ7"
- note added: "USB2_D+"
- note added: "USB2_D-"
- note added: "USB_OTG_FS_ID"
- note added: "USB_OTG_VBUS"
- note removed: "IGB_PREV"
- note removed: "TDM Mode"
- moved on the sheet: C1, C10, C11, C12, C13, C14, C15, C16, C17, C18, C20, C21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

Commit message: add CAN connector to core board
Parts:
- removed J2: VBUS_CON, Connector_Molex:Molex_KK-254_AE-6410-02A_1x02_P2.54mm_Vertical, symbol Connector_Generic:Conn_01x02
- removed R10, R11: 47, Resistor_SMD:R_0603_1608Metric, symbol Device:R
- removed R15, R16: 22, Resistor_SMD:R_0603_1608Metric, symbol Device:R
- added C4, C6: 100n, Capacitor_SMD:C_0805_2012Metric, symbol Device:C_Small
- added C7, C8: 47u, Capacitor_SMD:C_0805_2012Metric, symbol Device:C_Small
- added R13: 680, Resistor_SMD:R_0603_1608Metric, symbol Device:R
- added R22: 47k, Resistor_SMD:R_0402_1005Metric, symbol Device:R
- added R28, R29: 10k, Resistor_SMD:R_0402_1005Metric, symbol Device:R
- added R4: 0, Resistor_SMD:R_0603_1608Metric, symbol Device:R
- added U1: SIT1050T, Package_SO:SOP-8_3.9x4.9mm_P1.27mm, symbol SIT1050T:SIT1050T
- added U2: TPS2041B, Package_TO_SOT_SMD:SOT-23-5, symbol Power_Management:TPS2041B
- J10: value I2C_PREV -> CAN
- J18: renamed from J13; footprint Connector_Molex:Molex_KK-254_AE-6410-06A_1x06_P2.54mm_Vertical -> Connector_Molex:Molex_KK-254_AE-6410-12A_1x12_P2.54mm_Vertical; symbol Connector_Generic:Conn_01x06 -> Connector_Generic:Conn_01x12
- J2: renamed from J11; value I2C_NEXT -> I2C
- J6: value IGB2_PREV -> IGB_PREV
- J7: value IGB2_NEXT -> IGB_NEXT
- J8: value IGB3_NEXT -> IGB2_NEXT
- J9: value IGB4_NEXT -> IGB3_NEXT
- R1: renamed from R12; value 47 -> 22
- R14: value 22 -> 330
- R17: value 22 -> 680
- R2: renamed from R13; value 47 -> 22
- R32: renamed from R31; value 10k -> 47k
- R33: renamed from R32; value 10k -> 47k
- R34: renamed from R33; value 10k -> 47k
- R35: renamed from R34; value 10k -> 47k
- R39: renamed from R35; value 10k -> 47k
- R40: renamed from R36; value 10k -> 47k
- renumbered C6 to C10, C7 to C11, C8 to C12, C9 to C13, C10 to C14, C11 to C15, C12 to C16, C13 to C17, C14 to C18, C15 to C19, C16 to C20, C17 to C21, C18 to C22, C19 to C23, C20 to C24, C21 to C25, C22 to C26, C23 to C27, C4 to C5, C5 to C9, J12 to J11, J14 to J12, J15 to J13, J16 to J14, J17 to J15, J18 to J16, J19 to J17, J20 to J19, J21 to J20, J22 to J21, R7 to R10, R8 to R11, R9 to R12, R18 to R15, R19 to R16, R20 to R18, R21 to R19, R22 to R20, R23 to R21, R24 to R23, R25 to R24, R26 to R25, R27 to R26, R28 to R27, R1 to R3, R29 to R30, R30 to R31, R37 to R36, R38 to R37, R39 to R38, R40 to R41, R41 to R42, R42 to R43, R43 to R44, R44 to R45, R45 to R46, R46 to R47, R47 to R48, R48 to R49, R2 to R5, R49 to R50, R50 to R51, R51 to R52, R52 to R53, R53 to R54, R54 to R55, R55 to R56, R3 to R6, R4 to R7, R5 to R8, R6 to R9, U1 to U3, U2 to U4
Connections:
- net +3.3V: now also J4.4 (Pin_4), R22.1, R28.1, R29.1; no longer J4.3 (Pin_3)
- net +5V: now also J4.3 (Pin_3), C4.2, C7.1, U1.3 (VCC), U2.5 (IN); no longer J18.3 (Pin_3)
- net GND: now also J10.3 (Pin_3), J18.7 (Pin_7), J18.8 (Pin_8), R17.1, C4.1, C6.1, C7.2, C8.1, R13.2, U1.2 (GND), U2.2 (GND); no longer J10.2 (Pin_2), J4.4 (Pin_4)
- net I2C4_SCL: now also R29.2
- net I2C4_SDA: now also R28.2
- net USB1_D+: now also J18.1 (Pin_1); no longer R14.2
- net USB1_D-: now also J18.2 (Pin_2)
- net USB_OTG_FS_D+: now also J18.11 (Pin_11)
- net USB_OTG_FS_D-: now also J18.12 (Pin_12); no longer R17.2
- net VBUS: now also J18.10 (Pin_10), J18.9 (Pin_9), R4.2
- net at R14.1: now also U1.4 (RxD); no longer J18.1 (Pin_1)
- net USB2_D+: now reaches J18.5 (Pin_5)
- net USB2_D+: now also J11.27 (Pin_27)
- net USB2_D-: now reaches J18.6 (Pin_6)
- net USB2_D-: now also J11.25 (Pin_25); no longer R17.1
- net at J10.1 (Pin_1): now also U1.7 (CANH)
- net CAN1_TX: now reaches J3.29 (Pin_29)
- net CAN1_TX: now also U1.1 (TxD)
- net CAN1_RX: now reaches J3.31 (Pin_31)
- net CAN1_RX: now also R14.2, R17.2
- net CAN1_STBY: now reaches J3.33 (Pin_33)
- net CAN1_STBY: now also R13.1, U1.8 (STBY)
- net USB_OTG_FS_ID: now reaches J11.15 (Pin_15)
- net USB1_OC_DETECT: now reaches J11.17 (Pin_17)
- net USB1_OC_DETECT: now also R22.2, U2.3 (~{OC})
- net USB1_DRV: now reaches J11.23 (Pin_23)
- net USB1_DRV: now also U2.4 (~{EN})
- net at J11.9 (Pin_9): now also R4.1
- net I2C3_SCL: no longer names the net of J14.22 (Pin_22)
- net I2C3_SDA: no longer names the net of J11.40 (Pin_40)
- new net: C6.2, C8.2, J18.3 (Pin_3), U2.1 (OUT)
- new net: J10.2 (Pin_2), U1.6 (CANL)
- no-connect marks 114 -> 108
Other:
- note added: "500mA Limit"
- note added: "CAN Connector"
- note added: "MIDI1"
- note added: "MIDI2"
- note removed: "IGB_NEXT"
- note removed: "MIDI_IN_OUT"
- note removed: "USB2_D+"
- note removed: "USB2_D-"
- note removed: "USB_OTG_FS_ID"
- moved on the sheet: J2, J21, J6, J7, J8, J9, R1, R10, R11, R12, R2, R30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

Commit message: change header pin assignment for core board
Parts:
- removed R53, R54, R55, R56: 0, Resistor_SMD:R_0603_1608Metric, symbol Device:R
- added C10: 100n, Capacitor_SMD:C_0402_1005Metric, symbol Device:C_Small
- renumbered C10 to C11, C11 to C18, C18 to C19, C19 to C20, C20 to C21, C21 to C22, C22 to C23, C23 to C24, C24 to C25, C25 to C26, C26 to C27, C27 to C28, J11 to J10, J12 to J11, J13 to J12, J14 to J13, J15 to J14, J16 to J15, J17 to J16, J18 to J17, J19 to J18, J2 to J19, J3 to J2, J4 to J3, J5 to J4, J6 to J5, J7 to J6, J8 to J7, J9 to J8, J10 to J9, R3 to R1, R12 to R10, R13 to R11, R14 to R12, R15 to R13, R16 to R14, R17 to R15, R18 to R16, R19 to R17, R20 to R18, R21 to R19, R4 to R2, R22 to R20, R23 to R21, R24 to R22, R25 to R23, R26 to R24, R30 to R25, R27 to R26, R31 to R27, R1 to R28, R2 to R29, R5 to R3, R28 to R30, R29 to R31, R36 to R32, R37 to R33, R38 to R34, R39 to R35, R35 to R36, R41 to R37, R42 to R38, R40 to R39, R6 to R4, R33 to R40, R32 to R41, R34 to R42, R7 to R5, R8 to R6, R9 to R7, R10 to R8, R11 to R9
Connections:
- net CONF_BIT3 is gone; now on net LCD_TP_RST: J20.12 (Pin_12)
- net +3.3V: now also C10.2
- net GND: now also J3.11 (Pin_11), J3.17 (Pin_17), J4.21 (Pin_21), C10.1; no longer J3.12 (Pin_12), J3.23 (Pin_23), J3.7 (Pin_7)
- net GPIO_CLOCK_OUT: now also J3.22 (Pin_22); no longer J4.22 (Pin_22)
- net GPIO_RESET_OUT: now also J3.23 (Pin_23); no longer J4.23 (Pin_23)
- net I2C1_SCL: now also J18.11 (Pin_11), J21.11 (Pin_11), R27.2; no longer J4.16 (Pin_16)
- net I2C1_SDA: now also J18.12 (Pin_12), J21.10 (Pin_10), R25.2; no longer J4.15 (Pin_15)
- net I2C6_SCL: now also J4.22 (Pin_22); no longer J18.11 (Pin_11), J21.11 (Pin_11), R27.2
- net I2C6_SDA: now also J4.23 (Pin_23); no longer J18.12 (Pin_12), J21.10 (Pin_10), R25.2
- net LCD_BL: now also J20.26 (Pin_26); no longer J20.21 (Pin_21)
- net LCD_DC: now also J20.32 (Pin_32); no longer J20.20 (Pin_20)
- net LCD_RST: now also J20.28 (Pin_28); no longer J20.23 (Pin_23)
- net LCD_TP_INT: now also J20.14 (Pin_14); no longer J20.25 (Pin_25)
- net LCD_TP_RST: no longer J20.27 (Pin_27)
- net SDMMC3_CK: now also J4.19 (Pin_19); no longer J3.17 (Pin_17)
- net SDMMC3_CMD: now also J4.20 (Pin_20); no longer J3.18 (Pin_18)
- net SDMMC3_D0: now also J4.15 (Pin_15); no longer J3.13 (Pin_13)
- net SDMMC3_D1: now also J4.16 (Pin_16); no longer J3.14 (Pin_14)
- net SDMMC3_D2: now also J4.17 (Pin_17); no longer J3.15 (Pin_15)
- net SDMMC3_D3: now also J4.18 (Pin_18); no longer J3.16 (Pin_16)
- net SPI2_MISO: now also J3.20 (Pin_20); no longer J3.21 (Pin_21)
- net SPI2_MOSI: now also J3.19 (Pin_19); no longer J3.20 (Pin_20)
- net SPI2_NSS: now also J3.18 (Pin_18); no longer J3.19 (Pin_19)
- net SPI2_SCK: now also J3.21 (Pin_21); no longer J3.22 (Pin_22)
- net SPI4_GPIO_CS1: now also J3.12 (Pin_12); no longer J4.17 (Pin_17)
- net SPI4_MISO: now also J3.15 (Pin_15); no longer J4.20 (Pin_20)
- net SPI4_MOSI: now also J3.14 (Pin_14); no longer J4.19 (Pin_19)
- net SPI4_NSS: now also J3.13 (Pin_13); no longer J4.18 (Pin_18)
- net SPI4_SCK: now also J3.16 (Pin_16); no longer J4.21 (Pin_21)
- net USART1_RX: now also J3.7 (Pin_7); no longer J3.8 (Pin_8)
- net USART1_TX: now also J3.8 (Pin_8); no longer J3.9 (Pin_9)
- net USART3_RX: now also J3.9 (Pin_9); no longer J3.10 (Pin_10)
- net USART3_TX: now also J3.10 (Pin_10); no longer J3.11 (Pin_11)
- net CONF_BIT0: no longer names the net of J20.6 (Pin_6)
- net CONF_BIT1: no longer names the net of J20.8 (Pin_8)
- net CONF_BIT2: no longer names the net of J20.10 (Pin_10)
- no-connect marks 108 -> 112
Other:
- note removed: "Config"
- note removed: "Pull Ups"
- moved on the sheet: C18, C9, J19, J21, R25, R27, R28, R29, R30, R31, R35, R36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

Commit message: update core board sch&pcb
Parts:
- C4, C6: footprint Capacitor_SMD:C_0805_2012Metric -> Capacitor_SMD:C_0402_1005Metric
Connections:
- net GPIO_CLOCK_OUT: now also J2.37 (Pin_37); no longer J11.18 (Pin_18)
- net GPIO_RESET_OUT: now also J2.39 (Pin_39); no longer J11.20 (Pin_20)
- net I2C1_SDA: now also J20.36 (Pin_36); no longer J20.40 (Pin_40)
- net LCD_TP_INT: now also J20.12 (Pin_12); no longer J20.14 (Pin_14)
- net LCD_TP_RST: now also J20.10 (Pin_10); no longer J20.12 (Pin_12)
- net SPI2_MISO: now also J2.30 (Pin_30)
- net SPI2_MOSI: now also J2.40 (Pin_40); no longer J10.30 (Pin_30)
- net USART1_RX: now also R3.2; no longer J3.7 (Pin_7)
- net USART1_TX: now also R4.2; no longer J3.8 (Pin_8)
- net USART2_RX: now also R8.2; no longer R6.2
- net USART2_TX: now also R7.2; no longer R5.2
- net USART3_RX: now also R6.2; no longer J3.9 (Pin_9)
- net USART3_TX: now also R5.2; no longer J3.10 (Pin_10)
- net USART4_RX: now also J3.9 (Pin_9); no longer R3.2
- net USART4_TX: now also J3.10 (Pin_10); no longer R4.2
- net USART6_RX: now also R10.2; no longer R8.2
- net USART6_TX: now also R9.2; no longer R7.2
- net USB1_D+: now also J17.5 (Pin_5); no longer J17.1 (Pin_1)
- net USB1_D-: now also J17.6 (Pin_6); no longer J17.2 (Pin_2)
- net USB2_D+: now also J17.1 (Pin_1); no longer J17.5 (Pin_5)
- net USB2_D-: now also J17.2 (Pin_2); no longer J17.6 (Pin_6)
- net SPI6_MISO: now reaches J2.19 (Pin_19)
- net SPI6_MISO: now also J3.15 (Pin_15)
- net SPI6_NSS: now reaches J2.23 (Pin_23)
- net SPI6_NSS: now also J3.13 (Pin_13)
- net SPI6_MOSI: now reaches J2.24 (Pin_24)
- net SPI6_MOSI: now also J3.14 (Pin_14)
- net GPIO1: now reaches J2.25 (Pin_25)
- net GPIO1: now also J3.12 (Pin_12)
- net SPI6_SCK: now reaches J2.26 (Pin_26)
- net SPI6_SCK: now also J3.16 (Pin_16)
- net SPI2_CS_GPIO: now reaches J2.35 (Pin_35)
- net SPI2_CS_GPIO: now also J3.18 (Pin_18)
- net UART8_RX: now reaches J20.15 (Pin_15)
- net UART8_RX: now also J3.7 (Pin_7)
- net SPI2_NSS: no longer names the net of J16.28 (Pin_28)
- net SPI2_NSS: no longer J3.18 (Pin_18)
- net SPI4_GPIO_CS1: no longer names the net of J16.25 (Pin_25)
- net SPI4_GPIO_CS1: no longer J3.12 (Pin_12)
- net SPI4_MISO: no longer names the net of J16.29 (Pin_29)
- net SPI4_MISO: no longer J3.15 (Pin_15)
- net SPI4_MOSI: no longer names the net of J16.31 (Pin_31)
- net SPI4_MOSI: no longer J3.14 (Pin_14)
- net SPI4_NSS: no longer names the net of J11.40 (Pin_40)
- net SPI4_NSS: no longer J3.13 (Pin_13)
- net SPI4_SCK: no longer names the net of J16.27 (Pin_27)
- net SPI4_SCK: no longer J3.16 (Pin_16)
- net UART7_RX: no longer names the net of J13.33 (Pin_33)
- net UART7_RX: no longer R10.2
- net UART7_TX: no longer names the net of J13.35 (Pin_35)
- net UART7_TX: no longer R9.2
- net USB_OTG_FS_ID: no longer names the net of J10.15 (Pin_15)
- new net UART8_TX: J20.14 (Pin_14), J3.8 (Pin_8)
Other:
- note added: "CTRL_MCU_SPI"
- note added: "PA1/UART4_RX"
- note added: "PA2/USART2_TX"
- note added: "PA5/SPI1_SCK"
- note added: "PA6/SPI1_MISO"
- note added: "PA7/SPI1_MOSI/SPI6_MOSI"
- note added: "PB11/I2C2_SDA/USART3_RX"
- note added: "PB2/USART1_RX/UART4_RX"
- note added: "PB8/I2C1_SCL/I2C4_SCL/UART4_RX"
- note added: "PB9/I2C1_SDA/I2C4_SDA/SPI2_NSS/UART4_TX"
- note added: "PC1/SPI2_MOSI"
- note added: "PC2/SPI2_MISO"
- note added: "PD10/SPI3_MISO"
- note added: "PD13/I2C1_SDA/I2C4_SDA"
- note added: "PE11/SPI4_NSS"
- note added: "PE12/SPI4_SCK"
- note added: "PE13/SPI4_MISO"
- note added: "PE14/SPI4_MOSI"
- note added: "PE2/I2C4_SCK/SPI4_SCK"
- note added: "PE7/UART7_RX"
- note added: "PE8/UART7_TX"
- note added: "PG11/USART1_TX/UART4_TX"
- note added: "PG12/SPI6_MISO"
- note added: "PG13/SPI6_SCK"
- note added: "PG14/SPI6_MOSI/USART6_TX"
- note added: "PG8/SPI6_NSS"
- note added: "PH11/I2C4_SCL/I2C1_SCL"
- note added: "PH12/I2C4_SDA/I2C1_SDA"
- note added: "PH14/UART4_RX"
- note added: "PI0/SPI2_NSS"
- note added: "PI3/SPI2_MOSI"
- note added: "PJ8/UART8_TX"
- note added: "PJ9/UART8_RX"
- note added: "USB_OTG_FS_ID"
- note removed: "CTRL_MCU1_2_SPI"
- note removed: "PA1/GRXD_CLK"
- note removed: "PA2"
- note removed: "PA5"
- note removed: "PA6"
- note removed: "PA7/GRXD_DV"
- note removed: "PB11/GTXD_EN"
- note removed: "PB8"
- note removed: "PB9"
- note removed: "PC1"
- note removed: "PC2/GTXD2"
- note removed: "PD10"
- note removed: "PD13"
- note removed: "PE11"
- note removed: "PE12"
- note removed: "PE13"
- note removed: "PE14"
- note removed: "PE2/GTXD3"
- note removed: "PE7"
- note removed: "PE8"
- note removed: "PG11"
- note removed: "PG12"
- note removed: "PG13/GTXD0"
- note removed: "PG14/GTXD1"
- note removed: "PG8"
- note removed: "PH11"
- note removed: "PH12"
- note removed: "PH14"
- note removed: "PI0"
- note removed: "PI3"
- note removed: "PJ8"
- note removed: "PJ9"
- moved on the sheet: C1, C3, J10, J11, J13, J16, J2, J20, R2, TP1, TP2, TP3
