File: hardware/pcb/projects/igb01_module/igb01_module_ctrl/igb01_module_ctrl.kicad_pcb (KiCad board)
At the start: 2 copper layers, 131 x 111.1 mm, 278 parts, among them J1 ST_JACK_MIDI_OUT, J10 JACK_MAIN_L_OUT, J11 JACK_MAIN_R_OUT, J12 ST_JACK_MIDI_IN, J13 JACK_RST_OUT, J14 JACK_CV_Y_IN, J15 JACK_CV_E_OUT, J16 JACK_CV_F_OUT, J17 JACK_CV_G_OUT, J18 JACK_CV_H_OUT, J19 JACK_RTN_L_IN, J2 JACK_CLK_OUT, J20 JACK_RTN_R_IN, J21 JACK_SND_L_OUT, J22 JACK_SND_R_OUT, J23 JTAG, J24 LEFT_CON, J25 RIGHT_CON, J26 Conn_01x02, J27 SWD_CON, J28 DISP_CON1, J29 Micro_SD_Card, J3 JACK_CV_X_IN, J30 Conn_01x03, J31 Conn_01x03, J32 Conn_01x03, J33 POWER_CON, J34 Conn_01x02, J4 JACK_CV_A_OUT, J5 JACK_CV_B_OUT, J6 JACK_CV_C_OUT, J7 JACK_CV_D_OUT, J8 JACK_EXT_L_IN, J9 JACK_EXT_R_IN, SW1 SW_Push_45deg, SW10 SW_Push_45deg, SW11 SW_Push_45deg, SW12 SW_Push_45deg, SW13 SW_Push_45deg, SW14 SW_Push_45deg, SW15 SW_Push_45deg, SW16 SW_Push_45deg, SW17 SW_Push_45deg, SW18 SW_Push_45deg, SW19 SW_Push_45deg, SW2 SW_Push_45deg, SW20 SW_Push_45deg, SW21 SW_Push_45deg, SW22 SW_Push_45deg, SW23 SW_Push_45deg, SW24 SW_Push_45deg, SW25 SW_Push_45deg, SW26 SW_Push_45deg, SW27 SW_Push_45deg, SW28 SW_Push_45deg, SW29 SW_Push_45deg, SW3 SW_Push_45deg, SW30 SW_Push_45deg, SW31 SW_Push_45deg, SW32 SW_Push_45deg, SW33 SW_Push_45deg, SW34 SW_Push_45deg, SW35 SW_Push_45deg, SW36 SW_Push_45deg, SW4 SW_Push_45deg, SW5 SW_Push_45deg, SW6 SW_Push_45deg, SW7 SW_Push_45deg, SW8 SW_Push_45deg, SW9 SW_Push_45deg, U1 TL074, U10 STM32G431RBTx, U11 TL074, U12 R-78B5.0-2.0, U13 LDK320-3.3V, U14 LDK320-3.3V, U15 LM4040DBZ-10, U2 TL074, U3 74AHCT1G125, U4 TLP2361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

Commit message: add production file for igb01 module ctrl board
Parts:
- added REF**: JLC_TOOL_HOLE, kicadlib:JLC_TOOL_HOLE, F.Cu at (177.5, 157.5)
- added REF**: JLC_TOOL_HOLE, kicadlib:JLC_TOOL_HOLE, F.Cu at (53.0, 52.0)
Other:
- board text added: "-12V"
- board text added: "NO:"
- board text added: "POWER"
- board text added: "RED"
- board text added: "TOOL"
