File: hardware/pcb/projects/igb01_module/igb01_module_led/igb01_module_led.kicad_sch (KiCad schematic)
At the start: 45 parts, among them J1 DISP_CON1, J2 Conn_01x03, J3 Conn_01x02, J4 Conn_01x03, J5 Conn_01x02, J6 Conn_01x03, U1 IS31FL3731-QF

Commit message: add schematic pdfs
Other:
- title: (none) -> igb module led
Changed lines of the file:
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@@
 	(generator_version "9.0")
 	(paper "A3")
+	(title_block
+		(title "igb module led")
+		(rev "0.1")
+	)
 	(rectangle
 		(start 452.12 220.98)
